File: HW3/ME433_chip_board/ME433_chip_board.sch (EAGLE design)
At the start: 25 parts

Commit message: Fixed missing capacitor
Parts:
- added C5: (no value), ME433:CAP0603-CAP
Connections:
- net 3.3V: now also C5.1
- net GND: now also C5.2
Changed lines of the file:
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@@
 <part name="GND12" library="ME433" deviceset="GND" device=""/>
 <part name="P+7" library="ME433" deviceset="3.3V" device=""/>
+<part name="C5" library="ME433" deviceset="CAP" device="0603-CAP"/>
+<part name="GND13" library="ME433" deviceset="GND" device=""/>
 </parts>
 <sheets>
@@
 <instance part="GND12" gate="1" x="-40.64" y="22.86"/>
 <instance part="P+7" gate="G$1" x="-40.64" y="55.88"/>
+<instance part="C5" gate="G$1" x="-38.1" y="-35.56"/>
+<instance part="GND13" gate="1" x="-38.1" y="-43.18"/>
 </instances>
 <busses>
@@
 <pinref part="GND12" gate="1" pin="GND"/>
 <wire x1="-40.64" y1="27.94" x2="-40.64" y2="25.4" width="0.1524" layer="91"/>
+</segment>
+<segment>
+<pinref part="GND13" gate="1" pin="GND"/>
+<pinref part="C5" gate="G$1" pin="2"/>
+<wire x1="-38.1" y1="-40.64" x2="-38.1" y2="-38.1" width="0.1524" layer="91"/>
 </segment>
 </net>
@@
 <wire x1="-22.86" y1="-27.94" x2="-38.1" y2="-27.94" width="0.1524" layer="91"/>
 <pinref part="P+2" gate="G$1" pin="3.3V"/>
-</segment>
-<segment>
+<pinref part="C5" gate="G$1" pin="1"/>
+<wire x1="-38.1" y1="-30.48" x2="-38.1" y2="-27.94" width="0.1524" layer="91"/>
+<junction x="-38.1" y="-27.94"/>
+</segment>
+<segment>
